File: Hardware/SPI Hub PCB KiCad files/SPI_Hub.kicad_sch (KiCad schematic)
At the start: 18 parts, among them J1 Conn_01x08_Pin, J2 Left Front, J3 Left Center, J4 Left Rear, J5 Right Front, J6 Right Center, J7 Right Rear, U1 74AHC595, U2 74HC14

Commit message: Updated KiCad schematic, tied unused Schmitt input to gnd
Connections:
- net GND: now also U2.13
- net cipo_peripheral: now reaches J2.4 (Pin_4), J3.4 (Pin_4), J4.4 (Pin_4), J5.4 (Pin_4), J6.4 (Pin_4), J7.4 (Pin_4), U2.1
- no-connect marks 8 -> 7
Changed lines of the file:
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@@
+	)
+	(junction
+		(at 71.12 110.49)
+		(diameter 0)
+		(color 0 0 0 0)
 	)
 	(junction
@@
 	)
 	(no_connect
-		(at 71.12 119.38)
-	)
-	(no_connect
 		(at 86.36 92.71)
 	)
@@
 		(pts
 			(xy 181.61 16.51) (xy 181.61 40.64)
+		)
+		(stroke
+			(width 0)
+			(type default)
+		)
+	)
+	(wire
+		(pts
+			(xy 71.12 110.49) (xy 71.12 119.38)
 		)
 		(stroke
@@
 		(effects
 			(font
+				(size 1.27 1.27)
+			)
+			(justify left bottom)
+		)
+	)
+	(label "cipo_peripheral"
+		(at 105.41 81.28 0)
+		(effects
+			(font
